File: ESP_PP_AI.kicad_sch (KiCad schematic)
At the start: 12 parts, among them IC1 LM66200DRLR, J1 TYPE-C-31-M-12, Q1 AO3401A, U1 ESP32-S3, U2 MCP23017-E/SO-ND, U3 TPS63020DSJR, U4 MCP73831-2ACI_MC, U5 USBLC6-2SC6

Commit message: added_loadsharing
Parts:
- removed U1: ESP32-S3, Package_DFN_QFN:QFN-56-1EP_7x7mm_P0.4mm_EP4x4mm, symbol MCU_Espressif:ESP32-S3
- added C1, C2: 4.7uF, symbol Device:C
- added C10: 100nF, symbol Device:C
- added C3: 0.1uF, symbol Device:C
- added C4, C5, C9: 10uF, symbol Device:C
- added C6, C7, C8: 22uF, symbol Device:C
- added D2: CHARG, symbol Device:LED
- added D3: BAT_PWR, symbol Device:LED
- added D4: PWR_FAIL, symbol Device:LED
- added J2: BAT_IN, symbol Connector_Generic:Conn_01x02
- added L1: 1.5uH, symbol Device:L
- added R10: 200, symbol Device:R
- added R11, R9: 10K, symbol Device:R
- added R12, R13: 22, symbol Device:R
- added R4: 1K, symbol Device:R
- added R5: 2K, symbol Device:R
- added R6: 150, symbol Device:R
- added R7: 1M, symbol Device:R
- added R8: 180K, symbol Device:R
- added SW1: SWITCH, symbol Switch:SW_SPST
- added U6: ESP32-S3-WROOM-1, RF_Module:ESP32-S3-WROOM-1, symbol RF_Module:ESP32-S3-WROOM-1
Connections:
- net USB_5V is gone; now on net VDD: D1.2 (A), Q1.2 (S), U5.5
- net D+: now also R13.1
- net D-: now also R12.1
- net GND: now also IC1.1 (GND@1), IC1.4 (ON), IC1.5 (GND@2), U3.15 (PGND), U3.2 (GND), U4.6 (VSS), U4.9 (EP), C1.2, C10.2, C2.2, C3.2, C4.2, C5.2, C6.2, C7.2, C8.2, C9.2, J2.1 (Pin_1), R11.2, R5.2, R8.2, R9.2, U6.1 (GND), U6.40 (GND), U6.41 (GND)
- net VDD: now also IC1.3 (VIN1), C1.1, D2.2 (A)
- net BAT_3V: now reaches U4.3 (VBAT), U4.4 (VBAT)
- net BAT_3V: now also IC1.6 (VIN2), C2.1, J2.2 (Pin_2)
- net at U4.5 (STAT): now also R4.2
- net at U4.8 (PROG): now also R5.1
- net V_SYS: now reaches IC1.2 (VOUT@1)
- net V_SYS: now also IC1.7 (VOUT@2), U3.10 (VIN_10), U3.11 (VIN_11), C4.1, C5.1, D4.2 (A), R10.1, R6.2
- net at IC1.8 (ST): now also D3.1 (K)
- net at U3.1 (VINA): now also C3.1
- net at U3.12 (EN): now also R9.1, SW1.2 (B)
- net at U3.13 (PS/SYNC): now also R11.1
- net at U3.14 (PG): now also D4.1 (K)
- net at U3.3 (FB): now also R7.2, R8.1
- net V_3V3: now reaches U3.4 (VOUT_4)
- net V_3V3: now also U3.5 (VOUT_5), C10.1, C6.1, C7.1, C8.1, C9.1, R7.1, U6.2 (3V3)
- net at U3.6 (L2_6): now also U3.7 (L2_7), L1.2
- net at U3.8 (L1_8): now also U3.9 (L1_9), L1.1
- new net: D3.2 (A), R6.1
- new net: R10.2, SW1.1 (A)
- new net: R12.2, U6.13 (USB_D-)
- new net: R13.2, U6.14 (USB_D+)
- new net: D2.1 (K), R4.1
- no-connect marks 0 -> 5
Other:
- note added: "BAT_CHG"
- note added: "BB_3V3"
- note added: "Battery Charging and Input Supply Switching"
- note added: "ESD"
- note added: "For 3.3v"
- note added: "RPP"
- note added: "Type-C"
- note added: "USB/BAT_SW"
- note added: "USB_LED"
- moved on the sheet: D1, IC1, J1, Q1, R1, R2, R3, U2, U3, U4, U5

Commit message: added esp
Parts:
- added C11: 1uF, symbol Device:C
- added CAM1: OV2640, OV2640:OV2640, symbol OV2640:OV2640
- added R14, R15: 10K, symbol Device:R
- added SW2: EN, symbol Switch:SW_Push
- added SW3: BOOT, symbol Switch:SW_Push
- added U1: XC6206P282MR, Package_TO_SOT_SMD:SOT-23-3, symbol Regulator_Linear:XC6206PxxxMR
- added U7: XC6206P122MR, Package_TO_SOT_SMD:SOT-23-3, symbol Regulator_Linear:XC6206PxxxMR
Connections:
- net GND: now also C11.1, SW2.1, SW3.1
- net V_3V3: now also R14.2, R15.2
- net BOOT: now reaches U6.27 (IO0)
- net BOOT: now also R15.1, SW3.2
- net EN: now reaches U6.3 (EN)
- net EN: now also C11.2, R14.1, SW2.2
- new net: CAM1.15 (DGND), CAM1.MT1 (DGND), CAM1.MT2 (DGND)
- no-connect marks 5 -> 6
Other:
- note added: "BOOT_BTN"
- note added: "Battery Charging And Input Supply Switching"
- note added: "EN_BTN"
- note added: "ESP32-S3-WROOM-N16R8"
- note added: "ESP32-S3-WROOM-N16R8 And Buttons"
- note added: "USB-C Power In with ESD And Reverse Polarity Protection"
- note removed: "Battery Charging and Input Supply Switching"
- note removed: "USB-C Power In with ESD and Reverse Polarity Protection"
- moved on the sheet: C10, C9, R12, R13, U2, U6

Commit message: added_cam
Parts:
- added C12, C15, C17, C19, C21, C23, C25, C26: 0.1uF, symbol Device:C
- added C13, C14, C16, C18: 1uF, symbol Device:C
- added C20, C22, C24: 4.7uF, symbol Device:C
- added R16, R19: 10K, symbol Device:R
- added R17, R18: 4.7K, symbol Device:R
- U1: value XC6206P282MR -> XC6206P282PR
- U7: value XC6206P122MR -> XC6206P152PR
Connections:
- net GND: now also CAM1.15 (DGND), CAM1.2 (AGND), CAM1.MT1 (DGND), CAM1.MT2 (DGND), U1.1 (GND), U7.1 (GND), C12.2, C13.2, C14.2, C15.2, C16.2, C17.2, C18.2, C19.2, C20.2, C21.2, C22.2, C23.2, C24.2, C25.2, C26.1, R16.1
- net V_3V3: now also U1.3 (VI), U7.3 (VI), C12.1, C13.1, C14.1, C15.1, R17.2, R18.2, R19.2
- net 2V8: now reaches U1.2 (VO)
- net 2V8: now also CAM1.11 (DOVDD), CAM1.4 (AVDD), C16.1, C17.1, C22.1, C23.1, C24.1, C25.1
- net 1V5: now reaches CAM1.10 (DVDD)
- net 1V5: now also U7.2 (VO), C18.1, C19.1, C20.1, C21.1
- net CAM_SDL: now reaches CAM1.3 (SIO_D)
- net CAM_SDL: now also R18.1
- net CAM_SCL: now reaches CAM1.5 (SIO_C)
- net CAM_SCL: now also R17.1
- net at CAM1.6 (RESET): now also C26.2, R19.1
- net at CAM1.8 (PWDN): now also R16.2
- no-connect marks 6 -> 8
Other:
- note added: "1.5V Supply"
- note added: "2.8V Supply"
- note added: "Decoupling Capacitor"
- moved on the sheet: CAM1, U1, U7

Commit message: fixxed camera
Parts:
- added C27: 15pF, symbol Device:C
- R17, R18: now not fitted
Connections:
- net GND: now also C27.2
- net IO16: now reaches CAM1.12 (DATA9)
- net IO16: now also U6.9 (IO16)
- net IO15: now reaches CAM1.13 (XCLK)
- net IO15: now also U6.8 (IO15)
- net IO17: now reaches CAM1.14 (DATA8)
- net IO17: now also U6.10 (IO17)
- net IO18: now reaches CAM1.16 (DATA7)
- net IO18: now also U6.11 (IO18)
- net IO13: now reaches CAM1.17 (PCLK)
- net IO13: now also U6.21 (IO13), C27.1
- net IO12: now reaches CAM1.18 (DATA6)
- net IO12: now also U6.20 (IO12)
- net IO11: now reaches CAM1.19 (DATA2)
- net IO11: now also U6.19 (IO11)
- net IO10: now reaches CAM1.20 (DATA5)
- net IO10: now also U6.18 (IO10)
- net IO9: now reaches CAM1.21 (DATA3)
- net IO9: now also U6.17 (IO9)
- net IO8: now reaches CAM1.22 (DATA4)
- net IO8: now also U6.12 (IO8)
- net IO6: now reaches CAM1.7 (VSYNC)
- net IO6: now also U6.6 (IO6)
- net IO7: now reaches CAM1.9 (HREF)
- net IO7: now also U6.7 (IO7)
- net GPIO14: now reaches U6.22 (IO14)
- net GPIO21: now reaches U6.23 (IO21)
- net GPIO47: now reaches U6.24 (IO47)
- net GPIO48: now reaches U6.25 (IO48)
- net GPIO38: now reaches U6.31 (IO38)
- net GPIO2: now reaches U6.38 (IO2)
- net GPIO1: now reaches U6.39 (IO1)
- net GPIO4: now reaches U6.4 (IO4)
- net GPIO5: now reaches U6.5 (IO5)
- no-connect marks 8 -> 17
Other:
- note added: "IOxx -> CAM GPIOxx -> DEVICE"
- note added: "JTAG"
- note added: "JTAG_STP"
- note added: "OV2640 Camera"
- note added: "OV2640 Camera and Supplies"
- note added: "STRP"
- note added: "UART"
- moved on the sheet: C12, C13, C14, C15, C16, C17, C18, C19, C20, C21, C22, C23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

Commit message: rwer
Other:
- note added: "JTAG_STRP"
- note removed: "JTAG_STP"
Changed lines of the file:
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@@
 		)
 	)
-	(text "JTAG_STP"
+	(text "JTAG_STRP"
 		(exclude_from_sim no)
-		(at 112.522 197.104 0)
+		(at 113.284 197.104 0)
 		(effects
 			(font
